File: battery_charging_devboard.kicad_pcb (KiCad board)
At the start: 2 copper layers, 33 parts, among them J1 Conn_01x02_Male, J2 USB_C_Receptacle_USB2.0, Q1 DMP3036SSD, Q5 DMP3036SSD, U1 BQ24725A, U2 CYPD3177

Commit message: Schematic completed. Started routing.
Parts:
- added BT1: 18650, User_Battery:Battery_18650, F.Cu at (233.3, -55.6)
- added BT2: 18650, User_Battery:Battery_18650, F.Cu at (233.3, -32.5)
- added BT3: 18650, User_Battery:Battery_18650, F.Cu at (233.3, -9.40)
- added C10: 0.1u, Capacitor_SMD:C_0805_2012Metric_Pad1.18x1.45mm_HandSolder, F.Cu at (263.4, 48.7)
- added C11: 0.1u, Capacitor_SMD:C_0805_2012Metric_Pad1.18x1.45mm_HandSolder, F.Cu at (108.3, 63.8)
- added C12: 0.1u, Capacitor_SMD:C_0805_2012Metric_Pad1.18x1.45mm_HandSolder, F.Cu at (263.4, 54.7)
- added C13: 0.1u, Capacitor_SMD:C_0805_2012Metric_Pad1.18x1.45mm_HandSolder, F.Cu at (268.3, 42.7)
- added C14: 2.2u, Capacitor_SMD:C_0805_2012Metric_Pad1.18x1.45mm_HandSolder, F.Cu at (104.0, 71.1)
- added C15: 0.1u, Capacitor_SMD:C_0805_2012Metric_Pad1.18x1.45mm_HandSolder, F.Cu at (125.2, 59.7)
- added C16: 0.01u, Capacitor_SMD:C_0805_2012Metric_Pad1.18x1.45mm_HandSolder, F.Cu at (158.8, 75.8)
- added C17: 0.1u, Capacitor_SMD:C_0805_2012Metric_Pad1.18x1.45mm_HandSolder, F.Cu at (131.9, 59.8)
- added C18: 0.047u, Capacitor_SMD:C_0805_2012Metric_Pad1.18x1.45mm_HandSolder, F.Cu at (127.4, 59.7)
- added C19: 0.1u, Capacitor_SMD:C_0805_2012Metric_Pad1.18x1.45mm_HandSolder, F.Cu at (133.3, 69.0)
- added C20: 10u, Capacitor_SMD:C_1206_3216Metric_Pad1.33x1.80mm_HandSolder, F.Cu at (146.0, 55.8)
- added C21: 10u, Capacitor_SMD:C_1206_3216Metric_Pad1.33x1.80mm_HandSolder, F.Cu at (149.0, 79.9)
- added C22: 0.1u, Capacitor_SMD:C_0805_2012Metric_Pad1.18x1.45mm_HandSolder, F.Cu at (133.3, 71.2)
- added C23: 10u, Capacitor_SMD:C_1206_3216Metric_Pad1.33x1.80mm_HandSolder, F.Cu at (146.0, 58.3)
- added C24: 10u, Capacitor_SMD:C_1206_3216Metric_Pad1.33x1.80mm_HandSolder, F.Cu at (149.0, 86.6)
- added C25: 0.1u, Capacitor_SMD:C_0805_2012Metric_Pad1.18x1.45mm_HandSolder, F.Cu at (243.4, 82.1)
- added C26: 220u, Capacitor_SMD:CP_Elec_8x10, F.Cu at (281.5, 46.1)
- added C27: 0.33u, Capacitor_SMD:C_0805_2012Metric_Pad1.18x1.45mm_HandSolder, F.Cu at (243.4, 85.1)
- added C28: 0.1u, Capacitor_SMD:C_0805_2012Metric_Pad1.18x1.45mm_HandSolder, F.Cu at (243.4, 88.1)
- added C29: 10u, Capacitor_SMD:C_1206_3216Metric_Pad1.33x1.80mm_HandSolder, F.Cu at (146.0, 71.1)
- added C30: 10u, Capacitor_SMD:C_1206_3216Metric_Pad1.33x1.80mm_HandSolder, F.Cu at (146.0, 73.7)
- added C31: 0.1u, Capacitor_SMD:C_0805_2012Metric_Pad1.18x1.45mm_HandSolder, F.Cu at (243.4, 91.2)
- added C8: 100p, Capacitor_SMD:C_0805_2012Metric_Pad1.18x1.45mm_HandSolder, F.Cu at (125.1, 80.4)
- added C9: 2200p, Capacitor_SMD:C_0805_2012Metric_Pad1.18x1.45mm_HandSolder, F.Cu at (263.4, 45.7)
- added D10: BAT54WS, Diode_SMD:D_SOD-323_HandSoldering, F.Cu at (62.2, 47.0)
- added D11: SBR8M, Diode_SMD:D_PowerDI-5, F.Cu at (37.2, 82.5)
- added D2: MMSZ4684-TP, Diode_SMD:D_SOD-123, F.Cu at (225.8, 97.5)
- added D3: BAT54C, Package_TO_SOT_SMD:SOT-23, F.Cu at (123.0, 55.4)
- added D4: BAT54WS, Diode_SMD:D_SOD-323_HandSoldering, F.Cu at (129.7, 59.7)
- added D5: LED, LED_SMD:LED_0805_2012Metric_Pad1.15x1.40mm_HandSolder, F.Cu at (238.7, 82.1)
- added D6: LED, LED_SMD:LED_0805_2012Metric_Pad1.15x1.40mm_HandSolder, F.Cu at (238.7, 85.2)
- added D7: LED, LED_SMD:LED_0805_2012Metric_Pad1.15x1.40mm_HandSolder, F.Cu at (238.7, 88.2)
- added D8: LED, LED_SMD:LED_0805_2012Metric_Pad1.15x1.40mm_HandSolder, F.Cu at (76.5, 91.9)
- added D9: LED, LED_SMD:LED_0805_2012Metric_Pad1.15x1.40mm_HandSolder, F.Cu at (238.7, 91.3)
- added J3: COMM_SELECT, Connector_PinHeader_2.54mm:PinHeader_2x06_P2.54mm_Vertical_SMD, F.Cu at (242.7, 71.9)
- added J4: DEBUG_CONN, Connector_PinHeader_2.54mm:PinHeader_1x04_P2.54mm_Horizontal, F.Cu at (225.2, 65.6)
- added J5: UART_CONN, Connector_PinHeader_2.54mm:PinHeader_1x04_P2.54mm_Horizontal, F.Cu at (225.2, 77.8)
- added J7: UART_SUPP, Connector_PinHeader_2.54mm:PinHeader_1x02_P2.54mm_Vertical_SMD_Pin1Left, F.Cu at (249.8, 90.6)
- added L2: 4.7u, Inductor_SMD:L_Bourns_SRN8040TA, F.Cu at (155.0, 65.6)
- added Q11: MUN5335DW1T2G, Package_TO_SOT_SMD:SOT-363_SC-70-6_Handsoldering, F.Cu at (128.9, 53.9)
- added R19: 50k, Resistor_SMD:R_0805_2012Metric_Pad1.20x1.40mm_HandSolder, F.Cu at (73.3, 76.0)
- added R20: 4k, Resistor_SMD:R_0805_2012Metric_Pad1.20x1.40mm_HandSolder, F.Cu at (115.3, 69.0)
- added R21: 4k, Resistor_SMD:R_0805_2012Metric_Pad1.20x1.40mm_HandSolder, F.Cu at (111.3, 69.0)
- added R22: 430k, Resistor_SMD:R_0805_2012Metric_Pad1.20x1.40mm_HandSolder, F.Cu at (122.8, 80.3)
- added R23: 66.5k, Resistor_SMD:R_0805_2012Metric_Pad1.20x1.40mm_HandSolder, F.Cu at (122.8, 76.3)
- added R24: 10m, Resistor_SMD:R_1206_3216Metric_Pad1.30x1.75mm_HandSolder, F.Cu at (105.8, 63.6)
- added R25: 2, Resistor_SMD:R_0805_2012Metric_Pad1.20x1.40mm_HandSolder, F.Cu at (100.0, 71.2)
- added R26: 50k, Resistor_SMD:R_0805_2012Metric_Pad1.20x1.40mm_HandSolder, F.Cu at (129.7, 76.3)
- added R27: 316k, Resistor_SMD:R_0805_2012Metric_Pad1.20x1.40mm_HandSolder, F.Cu at (129.7, 80.4)
- added R28: 10k, Resistor_SMD:R_0805_2012Metric_Pad1.20x1.40mm_HandSolder, F.Cu at (115.3, 71.2)
- added R29: 10k, Resistor_SMD:R_0805_2012Metric_Pad1.20x1.40mm_HandSolder, F.Cu at (127.4, 76.3)
- added R30: 10k, Resistor_SMD:R_0805_2012Metric_Pad1.20x1.40mm_HandSolder, F.Cu at (127.4, 80.4)
- added R31: 50k, Resistor_SMD:R_0805_2012Metric_Pad1.20x1.40mm_HandSolder, F.Cu at (125.1, 76.3)
- added R32: 10, Resistor_SMD:R_0805_2012Metric_Pad1.20x1.40mm_HandSolder, F.Cu at (123.0, 59.6)
- added R33: 4k, Resistor_SMD:R_0805_2012Metric_Pad1.20x1.40mm_HandSolder, F.Cu at (133.3, 73.4)
- added R35: 10, Resistor_SMD:R_0805_2012Metric_Pad1.20x1.40mm_HandSolder, F.Cu at (137.4, 69.0)
- added R36: 10, Resistor_SMD:R_0805_2012Metric_Pad1.20x1.40mm_HandSolder, F.Cu at (137.4, 71.2)
- added R37: 660, Resistor_SMD:R_0805_2012Metric_Pad1.20x1.40mm_HandSolder, F.Cu at (220.5, 64.7)
- added R38: 660, Resistor_SMD:R_0805_2012Metric_Pad1.20x1.40mm_HandSolder, F.Cu at (220.5, 67.7)
- added R39: 660, Resistor_SMD:R_0805_2012Metric_Pad1.20x1.40mm_HandSolder, F.Cu at (220.5, 70.6)
- added R40: 2k, Resistor_SMD:R_0805_2012Metric_Pad1.20x1.40mm_HandSolder, F.Cu at (220.5, 73.6)
- added R41: 660, Resistor_SMD:R_0805_2012Metric_Pad1.20x1.40mm_HandSolder, F.Cu at (220.5, 76.5)
- added R42: 2k, Resistor_SMD:R_0805_2012Metric_Pad1.20x1.40mm_HandSolder, F.Cu at (220.5, 79.5)
- added R43: 2k, Resistor_SMD:R_0805_2012Metric_Pad1.20x1.40mm_HandSolder, F.Cu at (220.5, 82.4)
- added R44: 10k, Resistor_SMD:R_0805_2012Metric_Pad1.20x1.40mm_HandSolder, F.Cu at (220.5, 85.4)
- added R45: 58k, Resistor_SMD:R_0805_2012Metric_Pad1.20x1.40mm_HandSolder, F.Cu at (220.5, 88.3)
- added R46: 2k, Resistor_SMD:R_0805_2012Metric_Pad1.20x1.40mm_HandSolder, F.Cu at (72.5, 91.9)
- added R47: 10m, Resistor_SMD:R_1206_3216Metric_Pad1.30x1.75mm_HandSolder, F.Cu at (162.4, 65.9)
- added SW1: BAT_IND, Button_Switch_SMD:SW_SPST_PTS810, F.Cu at (249.2, 96.6)
- added TP2: HPI_INT, TestPoint:TestPoint_Pad_2.5x2.5mm, F.Cu at (268.2, 74.1)
- added TP3: debug_3V3, TestPoint:TestPoint_Pad_D1.0mm, F.Cu at (250.6, 64.8)
- added TP4: debug_swdio, TestPoint:TestPoint_Pad_D1.0mm, F.Cu at (250.6, 67.8)
- added TP5: debug_swclk, TestPoint:TestPoint_Pad_D1.0mm, F.Cu at (250.6, 70.9)
- added TP6: debug_gnd, TestPoint:TestPoint_Pad_D1.0mm, F.Cu at (250.6, 73.9)
- added TP7: ACOK_TP, TestPoint:TestPoint_Pad_2.5x2.5mm, F.Cu at (111.3, 72.0)
- added U10: RQ3E100BN, User_Mosfet:HSMT8, F.Cu at (145.8, 67.7)
- added U3: STM32F042F6Px, Package_SO:TSSOP-20_4.4x6.5mm_P0.65mm, F.Cu at (227.2, 91.8)
- added U4: T2N7002AK, Package_TO_SOT_SMD:SOT-23, F.Cu at (73.2, 79.0)
- added U5: L78L33_SO8, Package_SO:SOIC-8_3.9x4.9mm_P1.27mm, F.Cu at (250.1, 83.8)
- added U6: RQ3E100BN, User_Mosfet:HSMT8, F.Cu at (100.0, 67.9)
- added U7: RQ3E100BN, User_Mosfet:HSMT8, F.Cu at (100.0, 63.0)
- added U8: RQ3E100BN, User_Mosfet:HSMT8, F.Cu at (164.6, 75.0)
- added U9: RQ3E100BN, User_Mosfet:HSMT8, F.Cu at (146.0, 61.7)
- R10: value 660 -> 2k
- moved U1 101.2 mm to (124.0, 68.6)
- moved R1 74.3 mm to (77.3, 76.0), turned to 180 degrees
- moved R10 70.4 mm to (74.3, 83.1), turned to -90 degrees
- moved R12 63.0 mm to (82.2, 71.3), turned to 180 degrees
- moved R11 59.3 mm to (69.3, 76.0)
- moved R13 58.0 mm to (78.2, 71.3), turned to 180 degrees
- moved R2 57.4 mm to (59.6, 71.2)
- moved R3 57.2 mm to (63.5, 71.2)
- moved C4 57.0 mm to (68.3, 64.4), turned to 90 degrees
- moved C1 54.9 mm to (60.3, 61.0), turned to 90 degrees
- moved R5 54.4 mm to (63.5, 73.4)
- moved R4 54.3 mm to (59.6, 73.4)
- moved C2 54.3 mm to (62.5, 61.0), turned to 90 degrees
- moved C3 53.9 mm to (64.6, 61.0), turned to 90 degrees
- moved R8 53.4 mm to (59.7, 66.5)
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Connections:
- net I2C_CLK renamed HPI_CLK
- net I2C_SDA renamed HPI_SDA
- C1 pad 1: VREG_3V3 -> /usb_input/VDDD_3V3
- C2 pad 1: VREG_3V3 -> /usb_input/VDDD_3V3
- C3 pad 1: VREG_3V3 -> /usb_input/VDDD_3V3
- C5 pad 1: Net-(Q1A-D) -> USB_C_BUS
- C6 pad 1: Net-(Q1A-D) -> USB_C_BUS
- J1 pad 2: unconnected-(J1-Pin_2-Pad2) -> /usb_input/BACKUP_POWER
- J2 pad A4: Net-(Q1A-D) -> USB_C_BUS
- J2 pad A9: Net-(Q1A-D) -> USB_C_BUS
- J2 pad B4: Net-(Q1A-D) -> USB_C_BUS
- J2 pad B9: Net-(Q1A-D) -> USB_C_BUS
- Q1 pad 7: Net-(Q1A-D) -> USB_C_BUS
- Q1 pad 8: Net-(Q1A-D) -> USB_C_BUS
- Q5 pad 7: Net-(Q1A-D) -> USB_C_BUS
- Q5 pad 8: Net-(Q1A-D) -> USB_C_BUS
- R1 pad 1: VREG_3V3 -> /usb_input/VDDD_3V3
- R10 pad 1: Net-(D1-K) -> Net-(D1-A)
- R10 pad 2: GND -> USB_C_BUS
- R15 pad 1: Net-(Q1A-D) -> USB_C_BUS
- R18 pad 1: Net-(Q1A-D) -> USB_C_BUS
- R2 pad 1: VREG_3V3 -> /usb_input/VDDD_3V3
- R4 pad 1: VREG_3V3 -> /usb_input/VDDD_3V3
- R6 pad 1: VREG_3V3 -> /usb_input/VDDD_3V3
- R8 pad 1: unconnected-(R8-Pad1) -> /usb_input/VDDD_3V3
- U1 pad 1: unconnected-(U1-ACN-Pad1) -> POWER_SYSTEM
- U1 pad 10: unconnected-(U1-ILIM-Pad10) -> Net-(U1-ILIM)
- U1 pad 11: unconnected-(U1-BATDR-Pad11) -> Net-(U1-BATDR)
- U1 pad 12: unconnected-(U1-SRN-Pad12) -> Net-(U1-SRN)
- U1 pad 13: unconnected-(U1-SRP-Pad13) -> Net-(U1-SRP)
- U1 pad 14: Net-(U1-GND) -> GND
- U1 pad 15: unconnected-(U1-LODRV-Pad15) -> Net-(U1-LODRV)
- U1 pad 16: unconnected-(U1-REGN-Pad16) -> Net-(D4-A)
- U1 pad 17: unconnected-(U1-BTST-Pad17) -> Net-(D4-K)
- U1 pad 18: unconnected-(U1-HIDRV-Pad18) -> Net-(U1-HIDRV)
- U1 pad 19: unconnected-(U1-PHASE-Pad19) -> Net-(U1-PHASE)
- U1 pad 2: unconnected-(U1-ACP-Pad2) -> Net-(U1-ACP)
- U1 pad 20: unconnected-(U1-VCC-Pad20) -> Net-(U1-VCC)
- U1 pad 21: Net-(U1-GND) -> GND
- U1 pad 3: unconnected-(U1-CMSRC-Pad3) -> Net-(U1-CMSRC)
- U1 pad 4: unconnected-(U1-ACDRV-Pad4) -> Net-(U1-ACDRV)
- U1 pad 5: unconnected-(U1-ACOK-Pad5) -> Net-(U1-ACOK)
- U1 pad 6: unconnected-(U1-ACDET-Pad6) -> Net-(U1-ACDET)
- U1 pad 7: unconnected-(U1-IOUT-Pad7) -> uC_adc_Icharge
- U1 pad 8: unconnected-(U1-SDA-Pad8) -> I2C_SDA_CHRG
- U1 pad 9: unconnected-(U1-SCL-Pad9) -> I2C_CLK_CHRG
- U2 pad 18: Net-(Q1A-D) -> USB_C_BUS
- U2 pad 23: VREG_3V3 -> /usb_input/VDDD_3V3
- U2 pad 9: Net-(D1-A) -> Net-(U2-FAULT)
Routing:
- net USB_C_BUS: track 0.00 -> 41.4 mm
- net Net-(D10-A): track 0.00 -> 34.9 mm
- net Net-(U1-ACP): track 0.00 -> 29.6 mm
- net POWER_SYSTEM: track 0.00 -> 25.5 mm
- net Net-(C10-Pad1): track 0.00 -> 24.9 mm
- net Net-(C10-Pad2): track 0.00 -> 24.3 mm, vias 0 -> 2
- net Net-(C29-Pad2): track 0.00 -> 24.0 mm
- net /usb_input/VDDD_3V3: track 0.00 -> 20.4 mm
- net Net-(D10-K): track 0.00 -> 19.4 mm
- net Net-(U1-LODRV): track 0.00 -> 19.3 mm
- net V_USB_OUT: track 0.00 -> 19.2 mm
- net Net-(D4-A): track 0.00 -> 15.8 mm
- net Net-(U1-SRN): track 0.00 -> 15.5 mm
- net Net-(U1-ACOK): track 0.00 -> 14.0 mm
- net I2C_SDA_CHRG: track 0.00 -> 12.3 mm
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- added copper zone on B.Cu, net GND
- added copper zone on F.Cu, net GND
Other:
- board outline added: 129.2 x 89.8 mm

Commit message: Re-reouting the USB C CCX lines
Parts:
- added D12: BAT54WS, Diode_SMD:D_SOD-323_HandSoldering, F.Cu at (108.6, 89.8)
- added G***: LOGO, LOGO, F.Cu at (145.0, 105.0)
- added G***: LOGO, LOGO, B.Cu at (122.0, 82.0)
- added J7: OUT_SUP, Connector_PinHeader_2.54mm:PinHeader_1x02_P2.54mm_Vertical, F.Cu at (129.8, 124.6)
- added REF**: MountingHole_3mm_Pad_Via, MountingHole:MountingHole_3mm_Pad_Via, F.Cu at (152.0, 121.0)
- added REF**: MountingHole_3mm_Pad_Via, MountingHole:MountingHole_3mm_Pad_Via, F.Cu at (44.0, 121.0)
- added REF**: MountingHole_3mm_Pad_Via, MountingHole:MountingHole_3mm_Pad_Via, F.Cu at (44.0, 44.0)
- added REF**: MountingHole_3mm_Pad_Via, MountingHole:MountingHole_3mm_Pad_Via, F.Cu at (152.0, 44.0)
- BT1, BT2, BT3: moved to B.Cu
- moved TP1 208.6 mm to (59.6, 77.0)
- moved SW1 206.2 mm to (43.6, 81.0), turned to -90 degrees
- moved TP4 196.3 mm to (59.0, 116.4), turned to -90 degrees
- moved TP5 195.2 mm to (61.5, 116.4), turned to -90 degrees
- moved TP7 192.0 mm to (64.1, 116.4), turned to -90 degrees
- moved TP6 191.1 mm to (66.6, 116.4), turned to -90 degrees
- moved C10 186.6 mm to (77.2, 60.8), turned to 90 degrees
- moved C7 186.4 mm to (77.2, 54.0), turned to 90 degrees
- moved J4 182.2 mm to (45.8, 109.6), turned to 180 degrees
- moved D9 182.0 mm to (58.3, 107.0)
- moved J3 182.0 mm to (45.8, 96.2), turned to 180 degrees
- moved D8 181.4 mm to (58.3, 104.3)
- moved D7 181.2 mm to (58.3, 109.6)
- moved D10 180.9 mm to (58.2, 101.8)
- moved C14 174.9 mm to (93.6, 52.0), turned to -90 degrees
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- renumbered C2 to C1, C17 to C11, C19 to C12, C11 to C13, C13 to C14, C18 to C16, C29 to C17, C20 to C18, C30 to C19, C6 to C2, C23 to C20, C24 to C21, C21 to C22, C4 to C23, C27 to C24, C8 to C25, C16 to C26, C28 to C27, C22 to C28, C25 to C29, C1 to C3, C31 to C30, C26 to C31, C5 to C4, C7 to C5, C12 to C6, C9 to C7, C3 to C8, C14 to C9, D10 to D1, D7 to D10, D2 to D11, D11 to D2, D8 to D5, D1 to D6, D9 to D7, D6 to D8, D5 to D9, J4 to J3, J5 to J4, J3 to J5, J7 to J6, L2 to L1, Q5 to Q2, Q11 to Q3, R17 to R1, R24 to R10, R35 to R11, R47 to R12, R3 to R13, R46 to R14, R4 to R15, R6 to R16, R10 to R17, R8 to R18, R2 to R19, R16 to R2, R5 to R20, R11 to R21, R7 to R22, R1 to R23, R12 to R24, R28 to R25, R19 to R26, R9 to R27, R13 to R28, R36 to R29, R18 to R3, R27 to R30, R22 to R31, R23 to R32, R31 to R34, R30 to R35, R26 to R36, R29 to R37, R37 to R38, R38 to R39, R14 to R4, R39 to R40, R44 to R43, R45 to R44, R40 to R45, R43 to R46, R15 to R5, R25 to R6, R21 to R7, R20 to R8, R32 to R9, TP2 to TP1, TP7 to TP2, TP1 to TP3, TP6 to TP4, TP4 to TP5, TP3 to TP6, TP5 to TP7, U7 to U1, U5 to U10, U6 to U2, U1 to U3, U8 to U4, U9 to U5, U10 to U6, U2 to U7, U4 to U8, U3 to U9
Connections:
- BT1 pad 1: Net-(BT1-+) -> uC_adc_battery
- BT2 pad 1: uC_adc_battery -> Net-(BT1--)
- BT2 pad 2: Net-(BT1-+) -> Net-(BT2--)
- BT3 pad 1: Net-(BT1--) -> Net-(BT2--)
- J3 pad 2: /microcontroller/uC_swdio -> /microcontroller/uc_swclk
- J3 pad 3: /microcontroller/uc_swclk -> /microcontroller/uC_swdio
- J4 pad 1: Net-(J5-Pin_1) -> Net-(J4-Pin_1)
- J6 pad 1: Net-(J5-Pin_1) -> UART_SUPP_5V
- J6 pad 2: UART_SUPP_5V -> Net-(J4-Pin_1)
- R23 pad 1: /usb_input/VDDD_3V3 -> VREG_3V3
- U9 pad 11: /microcontroller/uC_sel_comms -> uC_bat_out_en
- U9 pad 3: uC_bat_out_en -> /microcontroller/uC_sel_comms
Routing:
- net POWER_SYSTEM: track 25.5 -> 207.1 mm, vias 0 -> 6
- net VREG_3V3: track 4.30 -> 177.3 mm, vias 0 -> 3
- net Net-(BT2--): track 0.00 -> 161.7 mm, vias 0 -> 4
- net Net-(BT1--): track 0.00 -> 148.0 mm, vias 0 -> 2
- net uC_adc_battery: track 0.00 -> 124.1 mm, vias 0 -> 4
- net /microcontroller/uC_uart_tx: track 0.00 -> 89.3 mm, vias 0 -> 2
- net /microcontroller/uC_uart_rx: track 0.00 -> 88.4 mm, vias 0 -> 2
- net Net-(J4-Pin_1): track 0.00 -> 87.5 mm
- net USB_C_BUS: track 41.4 -> 125.9 mm, vias 0 -> 2
- net V_USB_OUT: track 19.2 -> 102.7 mm, vias 0 -> 3
- net /microcontroller/uc_swclk: track 0.00 -> 69.9 mm
- net I2C_CLK_CHRG: track 6.03 -> 75.0 mm, vias 0 -> 4
- net USB_C_D-: track 0.00 -> 66.6 mm, vias 0 -> 5
- net /microcontroller/uC_swdio: track 0.00 -> 63.3 mm
- net USB_C_D+: track 1.80 -> 61.9 mm, vias 0 -> 4
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Other:
- board size 129.2 x 89.8 mm -> 119.5 x 87.5 mm
- board text added: "100%"
- board text added: "25%"
- board text added: "3V3"
- board text added: "50%"
- board text added: "75%"
- board text added: "BAT. CHARGE"
- board text added: "CHARGER COMS"
- board text added: "CLK"
- board text added: "CYPD3177 COMS"
- board text added: "CYPD3177 FAULT"
- board text added: "GND"
- board text added: "IO"
- board text added: "OUT +"
- board text added: "SEL CHARGER"
- board text added: "SEL CYPD3177"
- board text added: "U+ UART"
- board text added: "UART Rx"
- board text added: "UART Tx"
- board text added: "USB SAFE LINE"
- board text added: "battery_charging_devboard Daniel Adamkovic 22-Oct-2023 V1.0"
