File: hardware/battery_charger.kicad_sch (KiCad schematic)
At the start: 52 parts, among them J7 OUT_SUP, Q3 MUN5335DW1T2G, U1 BQ24725A, U1 RQ3E100BN, U2 RQ3E100BN, U4 RQ3E100BN, U5 RQ3E100BN, U6 RQ3E100BN

Commit message: Continuing routing
Parts:
- removed C31: 220u, Capacitor_SMD:CP_Elec_8x10, symbol Device:C_Polarized_Small
- added TPe (x18): TestPoint, TestPoint:TestPoint_Pad_D1.0mm, symbol Connector:TestPoint
- TP2: footprint TestPoint:TestPoint_Pad_2.5x2.5mm -> TestPoint:TestPoint_Pad_D1.5mm
- renumbered BT1 to BT200, BT2 to BT201, BT3 to BT202, D3 to D200, D4 to D201, L1 to L200, Q3 to Q200, U2 to U200, U1 to U201, U4 to U203, U5 to U204, U6 to U205
Connections:
- net I2C_CLK_CHRG: now also TPe.1
- net I2C_SDA_CHRG: now also TPe.1
- net POWER_SYSTEM: now also TPe.1
- net uC_adc_Icharge: now also TPe.1
- net uC_adc_battery: now also TPe.1
- net at C1.1, C1.1, R16.2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: now also TPe.1
- net at L200.2, R16.1, R16.2: now also TPe.1
- net at D200.2, Q200.3 (C2): now also TPe.1
- net at Q200.5 (B2), Q200.6 (C1): now also TPe.1
- net at C1.1, R16.1, U200.1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: now also TPe.1
- net at C1.2, C1.2, R16.1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: now also TPe.1
- net at R16.1, R16.1, U1.10 (ILIM): now also TPe.1
- net at C1.1, D201.2 (A), U1.16 (REGN): now also TPe.1
- net at U1.18 (HIDRV), U204.4: now also TPe.1
- net at C1.1, U1.19 (PHASE): now also C1.2, C1.2, L200.1, U204.1, U204.2, U204.3, U205.5, TPe.1
- net at C1.2, R16.2, U1.20 (VCC): now also TPe.1
- net at R16.1, R16.2, U1.6 (ACDET): now also TPe.1
- net at C1.2, R16.1, U203.4: now also TPe.1
Other:
- note removed: "Total of sys. capacitance Not required by charger IC"
- moved on the sheet: BT200, BT201, BT202, C1, L200, R16, U205
