File: hardware/microcontroller.kicad_sch (KiCad schematic)
At the start: 30 parts, among them J3 DEBUG_CONN, J4 UART_CONN, J5 COMM_SELECT, J6 UART_SUPP, SW1 BAT_IND, U10 L78L33_SO8, U9 STM32F042F6Px

Commit message: Continuing routing
Parts:
- removed J3: DEBUG_CONN, Connector_PinHeader_2.54mm:PinHeader_1x04_P2.54mm_Horizontal, symbol Connector:Conn_01x04_Pin
- removed J5: COMM_SELECT, Connector_PinHeader_2.54mm:PinHeader_2x06_P2.54mm_Vertical_SMD, symbol Connector_Generic:Conn_02x06_Odd_Even
- added SW301: SW_DIP_x06, Button_Switch_SMD:SW_DIP_SPSTx06_Slide_6.7x16.8mm_W8.61mm_P2.54mm_LowProfile, symbol Switch:SW_DIP_x06
- added TPe (x2): TestPoint, TestPoint:TestPoint_Pad_D1.0mm, symbol Connector:TestPoint
- J300: renamed from J6; footprint Connector_PinHeader_2.54mm:PinHeader_1x02_P2.54mm_Vertical_SMD_Pin1Left -> Jumper:SolderJumper-2_P1.3mm_Open_Pad1.0x1.5mm
- renumbered C24 to C300, C27 to C301, C29 to C302, C30 to C303, D11 to D301, D7 to D302, D9 to D303, D8 to D304, D10 to D305, J4 to J301, R44 to R300, R45 to R301, R43 to R302, R42 to R303, R41 to R304, R38 to R305, R39 to R306, R40 to R307, R46 to R308, SW1 to SW300, TP6 to TP300, TP5 to TP301, TP7 to TP302, TP4 to TP303, U10 to U300, U9 to U301
Connections:
- net HPI_CLK: now also SW301.1
- net HPI_SDA: now also SW301.2
- net I2C_CLK_CHRG: now also SW301.3
- net I2C_SDA_CHRG: now also SW301.4
- net uC_clk: now also SW301.10, SW301.12
- net uC_sda: now also SW301.11, SW301.9
- net uC_sel_comms: now also SW301.7, SW301.8, TPe.1
- net at C303.1, D301.1 (K), R300.1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: now also TPe.1
- net at R308.2: now also SW301.5
Other:
- moved on the sheet: R303, R308, SW300
