File: hardware/usb_input.kicad_sch (KiCad schematic)
At the start: 39 parts, among them J1 Conn_01x02_Male, J2 USB_C_Receptacle_USB2.0, Q1 DMP3036SSD, Q2 DMP3036SSD, U7 CYPD3177, U8 T2N7002AK

Commit message: Continuing routing
Parts:
- added TPe100, TPe101, TPe102, TPe103, TPe104, TPe105, TPe106, TPe107, TPe108, TPe109, TPe110, TPe111, TPe112, TPe113: TestPoint, TestPoint:TestPoint_Pad_D1.0mm, symbol Connector:TestPoint
- TP100: renamed from TP1; footprint TestPoint:TestPoint_Pad_2.5x2.5mm -> TestPoint:TestPoint_Pad_D1.5mm
- TP101: renamed from TP3; footprint TestPoint:TestPoint_Pad_2.5x2.5mm -> TestPoint:TestPoint_Pad_D1.5mm
- renumbered C2 to C100, C5 to C101, C3 to C102, C1 to C103, C8 to C104, C4 to C105, C23 to C106, D2 to D100, D5 to D102, D6 to D103, J2 to J100, J1 to J101, Q2 to Q100, Q1 to Q101, R5 to R100, R4 to R101, R14 to R102, R3 to R103, R2 to R104, R1 to R105, R24 to R106, R28 to R107, R23 to R108, R17 to R109, R21 to R110, R26 to R111, R19 to R112, R15 to R113, R16 to R114, R18 to R115, R13 to R116, R20 to R117, R22 to R118, R27 to R119, U7 to U100, U8 to U101
Connections:
- net CC1: now also TPe108.1
- net CC2: now also TPe109.1
- net HPI_CLK: now also TPe107.1
- net HPI_SDA: now also TPe110.1
- net USB_C_BUS: now also TPe105.1
- net USB_C_GPIO: now also TPe112.1
- net VDDD_3V3: now also TPe104.1
- net V_USB_OUT: now also U100.11 (VDC_OUT), TPe106.1
- net at R108.2, U100.10 (FLIP): now also TPe111.1
- net at R111.2, U100.9 (FAULT), U101.1 (G): now also TPe113.1
- net at Q101.2 (G), Q101.4 (G), R103.2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: now also TPe103.1
- net at D4.1 (K), Q100.1 (S), Q100.3 (S)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: now also TPe100.1
- net at C100.2, C101.2, D4.2 (A)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: now also TPe101.1
- net at Q101.1 (S), Q101.3 (S): now also TPe102.1
- no-connect marks 8 -> 7
Other:
- moved on the sheet: C102, C103, C104, J100
